Commit message: 在gazebo中完成了仿真的简单demo

File: src/carmodel/xacro/carmodel.urdf (robot description, URDF)
Before this commit: robot 123, 6 links, 5 joints
Links:
- link base_link: geometry collision mesh filename=package://carmodel/meshes/base_link.STL; visual mesh filename=package://carmodel/meshes/base_link.STL
- link radar_link: geometry collision mesh filename=package://carmodel/meshes/radar_link.STL; visual mesh filename=package://carmodel/meshes/radar_link.STL
- link wheel_left_back_link: geometry collision mesh filename=package://carmodel/meshes/wheel_left_back_link.STL; visual mesh filename=package://carmodel/meshes/wheel_left_back_link.STL
- link wheel_left_front_link: geometry collision mesh filename=package://carmodel/meshes/wheel_left_front_link.STL; visual mesh filename=package://carmodel/meshes/wheel_left_front_link.STL
- link wheel_right_back_link: geometry collision mesh filename=package://carmodel/meshes/wheel_right_back_link.STL; visual mesh filename=package://carmodel/meshes/wheel_right_back_link.STL
- link wheel_right_front_link: geometry collision mesh filename=package://carmodel/meshes/wheel_right_front_link.STL; visual mesh filename=package://carmodel/meshes/wheel_right_front_link.STL
Joints:
- joint radar_joint: axis 0 0 -1 -> 0 -1 0; type continuous -> fixed
- joint wheel_left_back_joint: origin xyz=-0.14497 -0.27038 0.044 rpy=0 0 0 -> xyz=-0.14497 0.27138 0.044 rpy=0 0 0
