Commit message: 完成了激光雷达的引入

File: src/carmodel/xacro/carassmble.xacro (robot description, xacro)
@@ -2,3 +2,4 @@
     <xacro:include filename="movecar.xacro"/>
     <xacro:include filename="carmodel.urdf"/>
+    <xacro:include filename="laser.xacro"/>
 </robot>

File: src/carmodel/xacro/carmodel.urdf (robot description, URDF)
Before this commit: robot carmodel, 6 links, 5 joints
Joints:
- joint radar_joint: origin xyz=0.0750275357424189 0 0.15 rpy=0 0 0 -> xyz=0.0750275357424189 0 0.3 rpy=0 0 0
