Commit message: 完成了正确打tf树，两车均可独立建图

File: src/carmodel/xacro/agv_0/laser.xacro (robot description, xacro)
@@ -56,5 +56,5 @@
 				<plugin name="gazebo_laser" filename="libgazebo_ros_laser.so">
 					<topicName>scan</topicName>
-					<frameName>agv0/laser_link</frameName>
+					<frameName>laser_link</frameName>
 				</plugin>
 			</sensor>

File: src/carmodel/xacro/agv_0/movecar.xacro (robot description, xacro)
@@ -30,5 +30,5 @@
             <rightRearJoint>wheel_right_back_link</rightRearJoint>
             <odometryRate>50.0</odometryRate>
-            <robotBaseFrame>agv0/base_link</robotBaseFrame>
+            <robotBaseFrame>base_link</robotBaseFrame>
             <broadcastTF>1</broadcastTF>
         </plugin>

File: src/carmodel/xacro/agv_1/carmodel.xacro (robot description, xacro)
@@ -1,5 +1,5 @@
 <?xml version="1.0"?>
 <robot name="carmodel" xmlns:xacro="http://ros.org/wiki/xacro">
-  <link name="base_link">
+  <link name="${ns}/base_link">
     <inertial>
       <origin
@@ -40,10 +40,10 @@
     </collision>
   </link>
-  <gazebo reference="base_link">
+  <gazebo reference="${ns}/base_link">
     <material>
       Gazebo/Grey
     </material>
   </gazebo>
-  <link name="wheel_left_front_link">
+  <link name="${ns}/wheel_left_front_link">
     <inertial>
       <origin
@@ -84,10 +84,10 @@
     </collision>
   </link>
-  <gazebo reference="wheel_left_front_link">
+  <gazebo reference="${ns}/wheel_left_front_link">
     <material>
       Gazebo/Yellow
     </material>
   </gazebo>
-  <joint name="wheel_left_front_joint"
+  <joint name="${ns}/wheel_left_front_joint"
     type="continuous">
     <origin
@@ -95,11 +95,11 @@
       rpy="0 0 0" />
     <parent
-      link="base_link" />
-    <child
-      link="wheel_left_front_link" />
+      link="${ns}/base_link" />
+    <child
+      link="${ns}/wheel_left_front_link" />
     <axis
       xyz="0 1 0" />
   </joint>
-  <link name="wheel_left_back_link">
+  <link name="${ns}/wheel_left_back_link">
     <inertial>
       <origin
@@ -140,10 +140,10 @@
     </collision>
   </link>
-  <gazebo reference="wheel_left_back_link">
+  <gazebo reference="${ns}/wheel_left_back_link">
     <material>
       Gazebo/Yellow
     </material>
   </gazebo>
-  <joint name="wheel_left_back_joint"
+  <joint name="${ns}/wheel_left_back_joint"
     type="continuous">
     <origin
@@ -151,11 +151,11 @@
       rpy="0 0 0" />
     <parent
-      link="base_link" />
-    <child
-      link="wheel_left_back_link" />
+      link="${ns}/base_link" />
+    <child
+      link="${ns}/wheel_left_back_link" />
     <axis
       xyz="0 1 0" />
   </joint>
-  <link name="wheel_right_back_link">
+  <link name="${ns}/wheel_right_back_link">
     <inertial>
       <origin
@@ -196,10 +196,10 @@
     </collision>
   </link>
-  <gazebo reference="wheel_right_back_link">
+  <gazebo reference="${ns}/wheel_right_back_link">
     <material>
       Gazebo/Yellow
     </material>
   </gazebo>
-  <joint name="wheel_right_back_joint"
+  <joint name="${ns}/wheel_right_back_joint"
     type="continuous">
     <origin
@@ -207,11 +207,11 @@
       rpy="0 0 0" />
     <parent
-      link="base_link" />
-    <child
-      link="wheel_right_back_link" />
+      link="${ns}/base_link" />
+    <child
+      link="${ns}/wheel_right_back_link" />
     <axis
       xyz="0 -1 0" />
   </joint>
-  <link name="wheel_right_front_link">
+  <link name="${ns}/wheel_right_front_link">
     <inertial>
       <origin
@@ -252,10 +252,10 @@
     </collision>
   </link>
-  <gazebo reference="wheel_right_front_link">
+  <gazebo reference="${ns}/wheel_right_front_link">
     <material>
       Gazebo/Yellow
     </material>
   </gazebo>
-  <joint name="wheel_right_front_joint"
+  <joint name="${ns}/wheel_right_front_joint"
     type="continuous">
     <origin
@@ -263,11 +263,11 @@
       rpy="0 0 0" />
     <parent
-      link="base_link" />
-    <child
-      link="wheel_right_front_link" />
+      link="${ns}/base_link" />
+    <child
+      link="${ns}/wheel_right_front_link" />
     <axis
       xyz="0 -1 0" />
   </joint>
-  <link name="radar_link">
+  <link name="${ns}/radar_link">
     <inertial>
       <origin
@@ -308,5 +308,5 @@
     </collision>
   </link>
-  <joint name="radar_joint"
+  <joint name="${ns}/radar_joint"
     type="fixed">
     <origin
@@ -314,7 +314,7 @@
       rpy="0 0 0" />
     <parent
-      link="base_link" />
-    <child
-      link="radar_link" />
+      link="${ns}/base_link" />
+    <child
+      link="${ns}/radar_link" />
     <axis
       xyz="0 -1 0" />

File: src/carmodel/xacro/agv_1/laser.xacro (robot description, xacro)
@@ -1,9 +1,9 @@
 <robot name="my_sensors" xmlns:xacro="http://wiki.ros.org/xacro">
     <!-- 雷达 -->
-    <gazebo reference="radar_link">
+    <gazebo reference="${ns}/radar_link">
       <sensor type="ray" name="rplidar">
         <!-- 坐标是0 z x-->
         <pose>0 0 0 0 0 0</pose>
-        <visualize>true</visualize>
+        <visualize>false</visualize>
         <update_rate>5.5</update_rate>
         <ray>
@@ -29,5 +29,5 @@
         <plugin name="gazebo_rplidar" filename="libgazebo_ros_laser.so">
           <topicName>scan</topicName>
-          <frameName>agv1/radar_link</frameName>
+          <frameName>${ns}/radar_link</frameName>
         </plugin>
       </sensor>

File: src/carmodel/xacro/agv_1/movecar.xacro (robot description, xacro)
@@ -15,20 +15,20 @@
     </xacro:macro>
     <!-- 每一个驱动轮都需要配置传动装置 -->
-    <xacro:joint_trans joint_name="wheel_left_front_link" />
-    <xacro:joint_trans joint_name="wheel_left_back_link" />
-    <xacro:joint_trans joint_name="wheel_right_front_link" />
-    <xacro:joint_trans joint_name="wheel_right_back_link" />
+    <xacro:joint_trans joint_name="${ns}/wheel_left_front_link" />
+    <xacro:joint_trans joint_name="${ns}/wheel_left_back_link" />
+    <xacro:joint_trans joint_name="${ns}/wheel_right_front_link" />
+    <xacro:joint_trans joint_name="${ns}/wheel_right_back_link" />
     <!-- 麦轮控制器 -->
     <gazebo>
         <plugin name="mecanum_controller" filename="libgazebo_ros_planar_move.so">
             <commandTopic>cmd_vel</commandTopic>
-            <odometryTopic>odom</odometryTopic>
-            <odometryFrame>odom</odometryFrame>
-            <leftFrontJoint>wheel_left_front_link</leftFrontJoint>
-            <rightFrontJoint>wheel_right_front_link</rightFrontJoint>
-            <leftRearJoint>wheel_left_back_link</leftRearJoint>
-            <rightRearJoint>wheel_right_back_link</rightRearJoint>
+            <odometryTopic>${ns}/odom</odometryTopic>
+            <odometryFrame>${ns}/odom</odometryFrame>
+            <leftFrontJoint>${ns}/wheel_left_front_link</leftFrontJoint>
+            <rightFrontJoint>${ns}/wheel_right_front_link</rightFrontJoint>
+            <leftRearJoint>${ns}/wheel_left_back_link</leftRearJoint>
+            <rightRearJoint>${ns}/wheel_right_back_link</rightRearJoint>
             <odometryRate>50</odometryRate>
-            <robotBaseFrame>agv1/base_link</robotBaseFrame>
+            <robotBaseFrame>${ns}/base_link</robotBaseFrame>
             <broadcastTF>1</broadcastTF>
         </plugin>
